File: schematic/rpi.sch (KiCad schematic (older format))
At the start: 39 parts, among them J6 USB_A, J7 RCJ-041, J8 Micro_SD_Card_Det, J9 HDMI_A, Q1 DMG1012T, Q2 DMG1012T, SW3 CLEAR, U10 ESD5384, U11 AP2331W, U9 RaspberryPi-CM3+L

Commit message: completed schematic
Parts:
- removed R11, R12, R13, R14, R28, R6: 2k, Resistor_SMD:R_0603_1608Metric_Pad0.98x0.95mm_HandSolder, symbol Device:R_Small
- removed R15, R16, R17, R18, R20, R21, R22, R23, R24, R25: 1K, Resistor_SMD:R_0603_1608Metric_Pad0.98x0.95mm_HandSolder, symbol Device:R_Small
- removed R26, R27: 100k, Resistor_SMD:R_0603_1608Metric_Pad0.98x0.95mm_HandSolder, symbol Device:R_Small
- added U11, U12, U13, U14, U15: TXB0104D, Package_SO:SOIC-14_3.9x8.7mm_P1.27mm, symbol Logic_LevelTranslator:TXB0104D
- R10, R7, R8, R9: value 2k -> 100k; footprint Resistor_SMD:R_0603_1608Metric_Pad0.98x0.95mm_HandSolder -> Resistor_SMD:R_0603_1608Metric
- renumbered C13 to C17, C14 to C18, C15 to C19, C16 to C20, C17 to C21, C18 to C22, J8 to J6, J6 to J8, R29 to R11, U10 to U16, U11 to U17, U9 to U6
Connections:
- net +3V3: now also U11.1 (VCCA), U12.1 (VCCA), U13.1 (VCCA), U14.1 (VCCA), U15.1 (VCCA)
- net +5V: now also U11.14 (VCCB), U12.14 (VCCB), U13.14 (VCCB), U14.14 (VCCB), U15.14 (VCCB)
- net CB2: now also U13.12 (B2)
- net CLEAR: now also U6.89 (GPIO27); no longer U6.5 (GPIO1)
- net DA: now also U15.10 (B4)
- net GND: now also R10.2, R7.2, R8.2, R9.2, U11.7 (GND), U12.7 (GND), U13.7 (GND), U14.7 (GND), U15.7 (GND); no longer R10.1, R7.1, R8.1, R9.1
- net PA0: now also U11.12 (B2); no longer U6.30 (GPIO29)
- net PA1: now also U11.11 (B3); no longer U6.34 (GPIO30)
- net PA2: now also U11.10 (B4); no longer U6.36 (GPIO31)
- net PA3: now also U14.13 (B1); no longer U6.46 (GPIO32)
- net PA4: now also U14.12 (B2); no longer U6.48 (GPIO33)
- net PA5: now also U14.11 (B3); no longer U6.52 (GPIO34)
- net PA6: now also U14.10 (B4); no longer U6.54 (GPIO35)
- net PB0: now also U12.13 (B1)
- net PB1: now also U12.12 (B2); no longer R7.2
- net PB2: now also U12.11 (B3); no longer R8.2
- net PB3: now also U12.10 (B4); no longer R9.2
- net PB4: now also U15.13 (B1); no longer R10.2
- net PB5: now also U15.12 (B2)
- net PB6: now also U15.11 (B3)
- net PHI2: now also U13.11 (B3); no longer U6.15 (GPIO4)
- net RDA: now also U13.13 (B1); no longer U6.82 (GPIO44)
- net RESET: now also U13.10 (B4)
- net STROBE: now also U11.13 (B1); no longer U6.28 (GPIO28)
- net HDMI_14: now reaches J9.14 (UTILITY)
- net RP_PA6: now reaches U6.58 (GPIO36)
- net RP_PA6: now also U14.5 (A4)
- net RP_PB0: now reaches U6.60 (GPIO37)
- net RP_PB0: now also U12.2 (A1)
- net RP_PB1: now reaches U6.64 (GPIO38)
- net RP_PB1: now also U12.3 (A2)
- net RP_PB2: now reaches U6.66 (GPIO39)
- net RP_PB2: now also U12.4 (A3)
- net RP_PB3: now reaches U6.70 (GPIO40)
- net RP_PB3: now also U12.5 (A4)
- net RP_OEB: now reaches U6.72 (GPIO41)
- net RP_OEB: now also U12.8 (OE), U15.8 (OE)
- net RP_RDA: now reaches U6.75 (GPIO22)
- net RP_RDA: now also U13.2 (A1)
- net RP_PB4: now reaches U6.76 (GPIO42)
- net RP_PB4: now also U15.2 (A1)
- net RP_CB2: now reaches U6.77 (GPIO23)
- net RP_CB2: now also U13.3 (A2)
- net RP_PB5: now reaches U6.78 (GPIO43)
- net RP_PB5: now also U15.3 (A2)
- net RP_PHI2: now reaches U6.81 (GPIO24)
- net RP_PHI2: now also U13.4 (A3)
- net RP_RST: now reaches U6.83 (GPIO25)
- net RP_RST: now also U13.5 (A4)
- net RP_DA: now reaches U6.84 (GPIO45)
- net RP_DA: now also R10.1, U15.5 (A4)
- net RP_OEC: now reaches U6.87 (GPIO26)
- net RP_OEC: now also U13.8 (OE)
- new net RP_OEA: U11.8 (OE), U14.8 (OE), U6.46 (GPIO32)
- new net RP_PA0: R9.1, U11.3 (A2), U6.30 (GPIO29)
- new net RP_PA1: U11.4 (A3), U6.34 (GPIO30)
- new net RP_PA2: U11.5 (A4), U6.36 (GPIO31)
- new net RP_PA3: U14.2 (A1), U6.48 (GPIO33)
- new net RP_PA4: U14.3 (A2), U6.52 (GPIO34)
- new net RP_PA5: U14.4 (A3), U6.54 (GPIO35)
- new net RP_PB6: R8.1, U15.4 (A3), U6.82 (GPIO44)
- new net RP_STB: R7.1, U11.2 (A1), U6.28 (GPIO28)
- no-connect marks 4 -> 3
Other:
- moved on the sheet: C17, C18, C19, J7, J8, J9, Q1, Q2, R11, SW3, U16, U6

Commit message: finished product v1
Parts:
- removed C17, C18, C19: 47uF, Capacitor_SMD:C_1206_3216Metric, symbol Device:C_Small
- removed C20: 4.7uF, Capacitor_SMD:C_0603_1608Metric_Pad1.08x0.95mm_HandSolder, symbol Device:C_Small
- removed C21, C22: 0.1uF, Capacitor_SMD:C_0603_1608Metric_Pad1.08x0.95mm_HandSolder, symbol Device:C_Small
- removed J6: Micro_SD_Card_Det, Connector_Card:microSD_HC_Molex_104031-0811, symbol Connector:Micro_SD_Card_Det
- removed J7: RCJ-041, CUI_RCJ-041, symbol RCJ-041:RCJ-041
- removed J8: USB_A, UJ2-AH-4-TH:CUI_UJ2-AH-4-TH, symbol Connector:USB_A
- removed J9: HDMI_A, 10029449-111RLF:10029449111RLF, symbol Connector:HDMI_A
- removed Q1, Q2: DMG1012T, Package_TO_SOT_SMD:SOT-523, symbol Transistor_FET:DMG1012T
- removed R10, R7, R8, R9: 100k, Resistor_SMD:R_0603_1608Metric, symbol Device:R_Small
- removed R11: 100k, Resistor_SMD:R_0603_1608Metric, symbol Device:R
- removed U16: ESD5384, SW-On-Semi:WLCSP9-1.14x1.14mm, symbol Power_Protection:ESD5384
- removed U17: AP2331W, Package_TO_SOT_SMD:SOT-23, symbol Power_Management:AP2331W
- removed U6: RaspberryPi-CM3+L, 1717254-4:17172544, symbol MCU_Module:RaspberryPi-CM3+L
- added U6: Raspberry_Pi_Zero, Connector:Raspberry_Pi_Zero, symbol Connector:Raspberry_Pi_Zero
Connections:
- net +3V3: now also U6.1 (3V3), U6.17 (3V3)
- net +5V: now also U6.2 (5V), U6.4 (5V)
- net CLEAR: now also U6.40 (GPIO21)
- net GND: now also U6.14 (GND), U6.20 (GND), U6.25 (GND), U6.30 (GND), U6.34 (GND), U6.39 (GND), U6.6 (GND), U6.9 (GND), U6.MT (Mount)
- net RP_CB2: now also U6.36 (GPIO16)
- net RP_DA: now also U6.32 (GPIO12)
- net RP_OEA: now also U6.10 (GPIO15)
- net RP_OEB: now also U6.24 (GPIO8)
- net RP_OEC: now also U6.37 (GPIO26)
- net RP_PA0: now also U6.5 (GPIO3)
- net RP_PA1: now also U6.8 (GPIO14)
- net RP_PA2: now also U6.7 (GPIO4)
- net RP_PA3: now also U6.12 (GPIO18)
- net RP_PA4: now also U6.13 (GPIO27)
- net RP_PA5: now also U6.15 (GPIO22)
- net RP_PA6: now also U6.16 (GPIO23)
- net RP_PB0: now also U6.19 (GPIO10)
- net RP_PB1: now also U6.21 (GPIO9)
- net RP_PB2: now also U6.22 (GPIO25)
- net RP_PB3: now also U6.23 (GPIO11)
- net RP_PB4: now also U6.26 (GPIO7)
- net RP_PB5: now also U6.29 (GPIO5)
- net RP_PB6: now also U6.31 (GPIO6)
- net RP_PHI2: now also U6.35 (GPIO19)
- net RP_RDA: now also U6.33 (GPIO13)
- net RP_RST: now also U6.38 (GPIO20)
- net RP_STB: now also U6.3 (GPIO2)
- no-connect marks 3 -> 2
Other:
- note added: "PWM on GPIO12, 18, 13, 19"
- moved on the sheet: SW3, U11, U12, U13, U14, U15

Commit message: finished apple 1
Connections:
- net GND: no longer U6.MT (Mount)
- no-connect marks 2 -> 3
Changed lines of the file:
@@
 	1650 3750 1950 3750
-Wire Wire Line
-	3100 4550 3200 4550
-Wire Wire Line
-	3200 4550 3200 4425
-Connection ~ 3100 4550
 Wire Wire Line
 	1650 3850 1950 3850
@@
 Wire Wire Line
 	3800 2875 3500 2875
+NoConn ~ 3200 4425
 $EndSCHEMATC
